File: matrix.kicad_sch (KiCad schematic)
At the start: 134 parts, among them SW10 #8, SW11 #9, SW12 #0, SW13 -_, SW14 =+, SW15 BSPC, SW16 DELETE, SW17 TAB, SW18 Q, SW19 W, SW2 ESC, SW20 E, SW21 R, SW22 T, SW23 Y, SW24 U, SW25 I, SW26 O, SW27 P, SW28 [{, SW29 ]}, SW3 #1, SW30 \|, SW31 PGUP, SW32 CAPS, SW33 A, SW34 S, SW35 D, SW36 F, SW37 G, SW38 H, SW39 J, SW4 #2, SW40 K, SW41 L, SW42 ;:, SW43 '", SW44 ENTER, SW45 PGDN, SW46 SHIFT, SW47 Z, SW48 X, SW49 C, SW5 #3, SW50 V, SW51 B, SW52 N, SW53 M, SW54 ,<, SW55 .>, SW56 /?, SW57 SHIFT, SW58 UP, SW59 FN, SW6 #4, SW60 CTRL, SW61 WIN, SW62 ALT, SW63 SPACE, SW64 ALT, SW65 CTRL, SW66 LEFT, SW67 DOWN, SW68 RIGHT, SW7 #5, SW8 #6, SW9 #7

Commit message: Footprint assignment
Parts:
- D1, D10, D11, D12, D13, D14, D15, D16, D17, D18, D19, D2, D20, D21, D22, D23, D24, D25, D26, D27, D28, D29, D3, D30, D31, D32, D33, D34, D35, D36, D37, D38, D39, D4, D40, D41, D42, D43, D44, D45, D46, D47, D48, D49, D5, D50, D51, D52, D53, D54, D55, D56, D57, D58, D59, D6, D60, D61, D62, D63, D64, D65, D66, D67, D7, D8, D9: footprint (none) -> Diode_SMD:D_SOD-123
- SW10, SW11, SW12, SW13, SW14, SW15, SW16, SW17, SW18, SW19, SW2, SW20, SW21, SW22, SW23, SW24, SW25, SW26, SW27, SW28, SW29, SW3, SW30, SW31, SW32, SW33, SW34, SW35, SW36, SW37, SW38, SW39, SW4, SW40, SW41, SW42, SW43, SW44, SW45, SW47, SW48, SW49, SW5, SW50, SW51, SW52, SW53, SW54, SW55, SW56, SW58, SW59, SW6, SW61, SW63, SW66, SW67, SW68, SW7, SW8, SW9: footprint (none) -> MX_Hotswap:MX-Hotswap-1U
- SW46: value SHIFT -> LSHIFT; footprint (none) -> MX_Hotswap:MX-Hotswap-1U
- SW57: value SHIFT -> RSHIFT; footprint (none) -> MX_Hotswap:MX-Hotswap-1U
- SW60: value CTRL -> LCTRL; footprint (none) -> MX_Hotswap:MX-Hotswap-1U
- SW62: value ALT -> LALT; footprint (none) -> MX_Hotswap:MX-Hotswap-1U
- SW64: value ALT -> RALT; footprint (none) -> MX_Hotswap:MX-Hotswap-1U
- SW65: value CTRL -> RCTRL; footprint (none) -> MX_Hotswap:MX-Hotswap-1U

Commit message: Assigned keysizes
Parts:
- SW15: footprint MX_Hotswap:MX-Hotswap-1U -> MX_Hotswap:MX-Hotswap-2U
- SW17, SW30: footprint MX_Hotswap:MX-Hotswap-1U -> MX_Hotswap:MX-Hotswap-1.5U
- SW32, SW57: footprint MX_Hotswap:MX-Hotswap-1U -> MX_Hotswap:MX-Hotswap-1.75U
- SW44, SW46: footprint MX_Hotswap:MX-Hotswap-1U -> MX_Hotswap:MX-Hotswap-2.25U
- SW60, SW61, SW62: footprint MX_Hotswap:MX-Hotswap-1U -> MX_Hotswap:MX-Hotswap-1.25U
- SW63: footprint MX_Hotswap:MX-Hotswap-1U -> MX_Hotswap:MX-Hotswap-6.25U
Changed lines of the file:
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@@
 			)
 		)
-		(property "Footprint" "MX_Hotswap:MX-Hotswap-1U"
+		(property "Footprint" "MX_Hotswap:MX-Hotswap-2U"
 			(at 246.38 26.67 0)
 			(hide yes)
@@
 			)
 		)
-		(property "Footprint" "MX_Hotswap:MX-Hotswap-1U"
+		(property "Footprint" "MX_Hotswap:MX-Hotswap-1.25U"
 			(at 68.58 109.22 0)
 			(hide yes)
@@
 			)
 		)
-		(property "Footprint" "MX_Hotswap:MX-Hotswap-1U"
+		(property "Footprint" "MX_Hotswap:MX-Hotswap-1.5U"
 			(at 35.56 46.99 0)
 			(hide yes)
@@
 			)
 		)
-		(property "Footprint" "MX_Hotswap:MX-Hotswap-1U"
+		(property "Footprint" "MX_Hotswap:MX-Hotswap-1.75U"
 			(at 35.56 67.31 0)
 			(hide yes)
@@
 			)
 		)
-		(property "Footprint" "MX_Hotswap:MX-Hotswap-1U"
+		(property "Footprint" "MX_Hotswap:MX-Hotswap-6.25U"
 			(at 133.35 109.22 0)
 			(hide yes)
@@
 			)
 		)
-		(property "Footprint" "MX_Hotswap:MX-Hotswap-1U"
+		(property "Footprint" "MX_Hotswap:MX-Hotswap-1.75U"
 			(at 231.14 88.9 0)
 			(hide yes)
@@
 			)
 		)
-		(property "Footprint" "MX_Hotswap:MX-Hotswap-1U"
+		(property "Footprint" "MX_Hotswap:MX-Hotswap-1.5U"
 			(at 246.38 46.99 0)
 			(hide yes)
@@
 			)
 		)
-		(property "Footprint" "MX_Hotswap:MX-Hotswap-1U"
+		(property "Footprint" "MX_Hotswap:MX-Hotswap-2.25U"
 			(at 35.56 88.9 0)
 			(hide yes)
@@
 			)
 		)
-		(property "Footprint" "MX_Hotswap:MX-Hotswap-1U"
+		(property "Footprint" "MX_Hotswap:MX-Hotswap-1.25U"
 			(at 52.07 109.22 0)
 			(hide yes)
@@
 			)
 		)
-		(property "Footprint" "MX_Hotswap:MX-Hotswap-1U"
+		(property "Footprint" "MX_Hotswap:MX-Hotswap-1.25U"
 			(at 35.56 109.22 0)
 			(hide yes)
@@
 			)
 		)
-		(property "Footprint" "MX_Hotswap:MX-Hotswap-1U"
+		(property "Footprint" "MX_Hotswap:MX-Hotswap-2.25U"
 			(at 246.38 67.31 0)
 			(hide yes)

Commit message: Update matrix layout
Parts:
- SW64, SW65: footprint MX_Hotswap:MX-Hotswap-1U -> MX_Hotswap:MX-Hotswap-1.25U
Changed lines of the file:
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@@
 			)
 		)
-		(property "Footprint" "MX_Hotswap:MX-Hotswap-1U"
+		(property "Footprint" "MX_Hotswap:MX-Hotswap-1.25U"
 			(at 214.63 109.22 0)
 			(hide yes)
@@
 			)
 		)
-		(property "Footprint" "MX_Hotswap:MX-Hotswap-1U"
+		(property "Footprint" "MX_Hotswap:MX-Hotswap-1.25U"
 			(at 198.12 109.22 0)
 			(hide yes)
