File: keyboard_v0.kicad_pcb (KiCad board)
At the start: 2 copper layers, 155 parts, among them J1 AVR-ISP-6, J3 UJ20-C-H-G-SMT-1-P16-TR, SW1 SW_RESET, SW10 #8, SW11 #9, SW12 #0, SW13 -_, SW14 =+, SW15 BSPC, SW16 DELETE, SW17 TAB, SW18 Q, SW19 W, SW2 ESC, SW20 E, SW21 R, SW22 T, SW23 Y, SW24 U, SW25 I, SW26 O, SW27 P, SW28 [{, SW29 ]}, SW3 #1, SW30 \|, SW31 PGUP, SW32 CAPS, SW33 A, SW34 S, SW35 D, SW36 F, SW37 G, SW38 H, SW39 J, SW4 #2, SW40 K, SW41 L, SW42 ;:, SW43 '", SW44 ENTER, SW45 PGDN, SW46 LSHIFT, SW47 Z, SW48 X, SW49 C, SW5 #3, SW50 V, SW51 B, SW52 N, SW53 M, SW54 ,<, SW55 .>, SW56 /?, SW57 RSHIFT, SW58 UP, SW59 FN, SW6 #4, SW60 LCTRL, SW61 WIN, SW62 LALT, SW63 SPACE, SW64 RALT, SW65 RCTRL, SW66 LEFT, SW67 DOWN, SW68 RIGHT, SW7 #5, SW8 #6, SW9 #7, U1 ATmega32U4-A, U2 USBLC6-2P6, Y1 Crystal_GND24_Small

Commit message: Update matrix layout
Parts:
- C1, C2, C3, C4, C5, C6, C7, C8, D1, D10, D11, D12, D13, D14, D15, D16, D17, D18, D19, D2, D20, D21, D22, D23, D24, D25, D26, D27, D28, D29, D3, D30, D31, D32, D33, D34, D35, D36, D37, D38, D39, D4, D40, D41, D42, D43, D44, D45, D46, D47, D48, D49, D5, D50, D51, D52, D53, D54, D55, D56, D57, D58, D59, D6, D60, D61, D62, D63, D64, D65, D66, D67, D7, D8, D9, F1, J1, J3, R1, R2, R3, R4, R5, R6, SW1, U1, U2, Y1: moved to B.Cu
- SW64, SW65: footprint MX_Hotswap:MX-Hotswap-1U -> MX_Hotswap:MX-Hotswap-1.25U
- moved SW16 267.3 mm to (337.0, 73.8)
- moved SW31 251.1 mm to (337.0, 92.9)
- moved SW45 234.5 mm to (337.0, 111.9)
- moved SW30 226.8 mm to (313.2, 92.9)
- moved SW59 217.8 mm to (337.0, 131.0)
- moved SW14 210.6 mm to (279.9, 73.8)
- moved SW12 203.7 mm to (241.8, 73.8)
- moved SW29 202.9 mm to (289.4, 92.9)
- moved SW68 202.4 mm to (337.0, 150.0)
- moved SW58 198.1 mm to (318.0, 131.0)
- moved SW13 192.6 mm to (260.8, 73.8)
- moved D15 189.9 mm to (342.4, 78.4), turned to 90 degrees
- moved D67 188.2 mm to (342.6, 154.8), turned to 90 degrees
- moved D30 185.9 mm to (342.6, 97.6), turned to 90 degrees
- moved SW67 185.5 mm to (318.0, 150.0)
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
Commit message: Added edge cuts
Parts:
- moved SW65 40.0 mm to (250.0, 114.3)
- moved SW68 40.0 mm to (319.1, 114.3)
- moved C2 40.0 mm to (166.7, 110.3)
- moved C3 40.0 mm to (166.7, 118.3)
- moved C5 40.0 mm to (181.0, 122.2)
- moved D13 40.0 mm to (267.3, 42.7)
- moved D42 40.0 mm to (262.7, 81.0)
- moved D64 40.0 mm to (256.4, 119.1)
- moved D65 40.0 mm to (286.5, 119.1)
- moved R3 40.0 mm to (170.9, 122.2)
- moved SW42 40.0 mm to (238.1, 76.2)
- moved SW44 40.0 mm to (288.1, 76.2)
- moved SW63 40.0 mm to (154.8, 114.3)
- moved SW64 40.0 mm to (226.2, 114.3)
- moved U1 40.0 mm to (176.2, 114.3)
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Other:
- board outline added: 304.8 x 100 mm

Commit message: Update edge cuts
Other:
- board size 304.8 x 100 mm -> 304.8 x 101.3 mm
Changed lines of the file:
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@@
 	)
 	(gr_line
-		(start 23.8125 122.2375)
+		(start 23.8125 123.496218)
 		(end 23.8125 30.1625)
 		(stroke
@@
 	)
 	(gr_arc
-		(start 25.4 123.825)
-		(mid 24.277468 123.360032)
-		(end 23.8125 122.2375)
+		(start 25.4 125.083718)
+		(mid 24.277468 124.61875)
+		(end 23.8125 123.496218)
 		(stroke
 			(width 0.05)
@@
 	)
 	(gr_line
-		(start 327.025 123.825)
-		(end 25.4 123.825)
+		(start 327.025 125.083718)
+		(end 25.4 125.083718)
 		(stroke
 			(width 0.05)
@@
 	(gr_line
 		(start 328.6125 30.1625)
-		(end 328.6125 122.2375)
+		(end 328.6125 123.496218)
 		(stroke
 			(width 0.05)
@@
 	)
 	(gr_arc
-		(start 328.6125 122.2375)
-		(mid 328.147532 123.360032)
-		(end 327.025 123.825)
+		(start 328.6125 123.496218)
+		(mid 328.147532 124.61875)
+		(end 327.025 125.083718)
 		(stroke
 			(width 0.05)

Commit message: Complete routing
Parts:
- moved C2 11.7 mm to (177.4, 105.6)
- moved SW1 11.3 mm to (213.1, 114.2), turned to 180 degrees
- moved C3 10.2 mm to (176.9, 119.1), turned to 90 degrees
- moved R6 9.49 mm to (196.8, 106.0)
- moved C8 9.33 mm to (186.2, 104.3)
- moved R3 9.27 mm to (180.2, 121.8)
- moved U1 9.27 mm to (185.5, 113.9)
- moved C1 9.26 mm to (188.2, 105.1)
- moved R5 9.15 mm to (184.0, 103.8)
- moved R4 9.12 mm to (182.0, 103.8)
- moved C6 9.04 mm to (201.8, 116.1), turned to 0 degrees
- moved Y1 9.02 mm to (197.3, 115.3)
- moved C7 8.99 mm to (201.8, 113.5)
- moved C5 8.75 mm to (189.7, 121.7)
- moved C4 8.39 mm to (196.0, 109.8), turned to -90 degrees
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Connections:
- J3 pad A6: Net-(J3-DP1) -> DP
- J3 pad A7: Net-(J3-DN1) -> DN
- J3 pad B6: Net-(J3-DP1) -> DP
- J3 pad B7: Net-(J3-DN1) -> DN
- R4 pad 1: Net-(J3-DN1) -> Net-(R4-Pad1)
- R5 pad 1: Net-(J3-DP1) -> Net-(R5-Pad1)
- U1 pad 36: col6 -> col5
- U1 pad 37: col5 -> col6
- U1 pad 38: row1 -> row4
- U1 pad 39: row4 -> row1
- U1 pad 40: row3 -> row2
- U1 pad 41: row2 -> row3
- U2 pad 1: Net-(U2-I/O1-Pad1) -> DN
- U2 pad 3: Net-(U2-I/O2-Pad3) -> DP
- U2 pad 4: Net-(U2-I/O2-Pad3) -> Net-(R5-Pad1)
- U2 pad 6: Net-(U2-I/O1-Pad1) -> Net-(R4-Pad1)
Routing:
- net row0: track 0.00 -> 362.0 mm, vias 0 -> 4
- net row1: track 0.00 -> 351.2 mm, vias 0 -> 2
- net row2: track 0.00 -> 325.0 mm, vias 0 -> 2
- net row3: track 0.00 -> 292.4 mm, vias 0 -> 2
- net row4: track 0.00 -> 291.3 mm, vias 0 -> 2
- net col0: track 0.00 -> 265.8 mm, vias 0 -> 1
- net GND: track 0.00 -> 253.0 mm, vias 0 -> 5
- net col1: track 0.00 -> 250.2 mm, vias 0 -> 1
- net col14: track 0.00 -> 226.8 mm, vias 0 -> 1
- net col2: track 0.00 -> 220.9 mm, vias 0 -> 1
- net col13: track 0.00 -> 214.3 mm, vias 0 -> 1
- net +5V: track 0.00 -> 210.0 mm, vias 0 -> 7
- net col12: track 0.00 -> 191.2 mm, vias 0 -> 1
- net col3: track 0.00 -> 176.7 mm, vias 0 -> 1
- net col4: track 0.00 -> 158.3 mm, vias 0 -> 1
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- added copper zone on F.Cu, net GND
