File: keyboard_v0.kicad_pcb (KiCad board)
At the start: 2 copper layers, 304.8 x 101.3 mm, 155 parts, among them J1 AVR-ISP-6, J3 UJ20-C-H-G-SMT-1-P16-TR, SW1 SW_RESET, SW10 #8, SW11 #9, SW12 #0, SW13 -_, SW14 =+, SW15 BSPC, SW16 DELETE, SW17 TAB, SW18 Q, SW19 W, SW2 ESC, SW20 E, SW21 R, SW22 T, SW23 Y, SW24 U, SW25 I, SW26 O, SW27 P, SW28 [{, SW29 ]}, SW3 #1, SW30 \|, SW31 PGUP, SW32 CAPS, SW33 A, SW34 S, SW35 D, SW36 F, SW37 G, SW38 H, SW39 J, SW4 #2, SW40 K, SW41 L, SW42 ;:, SW43 '", SW44 ENTER, SW45 PGDN, SW46 LSHIFT, SW47 Z, SW48 X, SW49 C, SW5 #3, SW50 V, SW51 B, SW52 N, SW53 M, SW54 ,<, SW55 .>, SW56 /?, SW57 RSHIFT, SW58 UP, SW59 FN, SW6 #4, SW60 LCTRL, SW61 WIN, SW62 LALT, SW63 SPACE, SW64 RALT, SW65 RCTRL, SW66 LEFT, SW67 DOWN, SW68 RIGHT, SW7 #5, SW8 #6, SW9 #7, U1 ATmega32U4-A, U2 USBLC6-2P6, Y1 Crystal_GND24_Small

Commit message: Added Jellyfish
Parts:
- added G***: LOGO, Personal:Jellyfish, F.Cu at (120.9, 111.0)
Changed lines of the file:
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@@
 		)
+	)
+	(footprint "Personal:Jellyfish"
+		(layer "F.Cu")
+		(at 120.904 110.998)
+		(property "Reference" "G***"
+			(at 0 0 0)
+			(layer "F.SilkS")
+			(hide yes)
+			(effects
+				(font
+					(size 1.5 1.5)
+					(thickness 0.3)
+				)
+			)
+		)
+		(property "Value" "LOGO"
+			(at 0.75 0 0)
+			(layer "F.SilkS")
+			(hide yes)
+			(effects
+				(font
+					(size 1.5 1.5)
+					(thickness 0.3)
+				)
+			)
+		)
+		(property "Datasheet" ""
+			(at 0 0 0)
+			(layer "F.Fab")
+			(hide yes)
+			(effects
+				(font
+					(size 1.27 1.27)
+				)
+			)
+		)
+		(property "Description" ""
+			(at 0 0 0)
+			(layer "F.Fab")
+			(hide yes)
+			(effects
+				(font
+					(size 1.27 1.27)
+				)
+			)
+		)
+		(attr board_only exclude_from_pos_files exclude_from_bom)
+		(duplicate_pad_numbers_are_jumpers no)
+		(fp_poly
+			(pts
+				(xy 1.623382 -12.234718) (xy 3.982279 -11.714883) (xy 6.223632 -10.721477) (xy 8.28928 -9.256732)
+				(xy 8.683602 -8.90047) (xy 10.088216 -7.305684) (xy 10.988228 -5.67359) (xy 11.392077 -4.05133)
+				(xy 11.308202 -2.486045) (xy 10.745043 -1.024876) (xy 9.711038 0.285036) (xy 8.214626 1.396548)
+				(xy 6.713954 2.102273) (xy 5.967119 2.447594) (xy 5.464766 2.797393) (xy 5.347261 2.969405) (xy 5.452495 3.506719)
+				(xy 5.860826 4.272818) (xy 6.478546 5.146396) (xy 7.211949 6.006148) (xy 7.967328 6.730768) (xy 8.590947 7.168424)
+				(xy 9.495782 7.732835) (xy 9.916503 8.230265) (xy 9.885367 8.709395) (xy 9.747635 8.914086) (xy 9.204984 9.201405)
+				(xy 8.462506 9.087161) (xy 7.587136 8.626798) (xy 6.645808 7.875759) (xy 5.705456 6.889488) (xy 4.833014 5.72343)
+				(xy 4.095415 4.433029) (xy 3.943997 4.106706) (xy 3.534023 3.365906) (xy 3.134631 2.954847) (xy 2.991952 2.910416)
+				(xy 2.771405 2.983205) (xy 2.666964 3.274269) (xy 2.662104 3.892653) (xy 2.719693 4.706875) (xy 3.067638 6.767349)
+				(xy 3.723421 8.6384) (xy 4.592921 10.114054) (xy 5.100485 10.850378) (xy 5.260142 11.340898) (xy 5.094271 11.717836)
+				(xy 4.896116 11.90515) (xy 4.374585 12.052814) (xy 3.786475 11.757609) (xy 3.171258 11.095097) (xy 2.568402 10.140841)
+				(xy 2.017379 8.970404) (xy 1.557659 7.659348) (xy 1.228711 6.283236) (xy 1.070007 4.917629) (xy 1.061473 4.564062)
+				(xy 1.043735 3.756123) (xy 0.945912 3.344112) (xy 0.693968 3.194826) (xy 0.289411 3.174999) (xy -0.162599 3.212459)
+				(xy -0.416981 3.412672) (xy -0.563674 3.90739) (xy -0.658819 4.564062) (xy -1.012182 6.596256) (xy -1.512793 8.479575)
+				(xy -2.123404 10.106817) (xy -2.806767 11.370778) (xy -3.196785 11.868679) (xy -3.807951 12.307087)
+				(xy -4.416785 12.415053) (xy -4.858016 12.176074) (xy -4.930166 12.041767) (xy -4.876019 11.619181)
+				(xy -4.577661 10.942925) (xy -4.250074 10.393311) (xy -3.34244 8.621941) (xy -2.690688 6.467033)
+				(xy -2.393629 4.700247) (xy -2.298067 3.755705) (xy -2.320232 3.219756) (xy -2.503431 2.977083)
+				(xy -2.890969 2.912372) (xy -3.065784 2.910416) (xy -3.525852 3.044722) (xy -3.786835 3.535405)
+				(xy -3.843805 3.770312) (xy -4.340524 5.179634) (xy -5.172362 6.590708) (xy -6.196972 7.778163)
+				(xy -6.581004 8.103992) (xy -7.565464 8.749238) (xy -8.28922 8.966553) (xy -8.792904 8.762993) (xy -8.968063 8.518556)
+				(xy -9.106701 8.05311) (xy -8.911302 7.644907) (xy -8.314329 7.188965) (xy -7.985709 6.991531) (xy -7.383037 6.512903)
+				(xy -6.722925 5.799311) (xy -6.121495 5.002695) (xy -5.694869 4.274993) (xy -5.556251 3.812736)
+				(xy -5.465144 3.272203) (xy -5.406042 3.091426) (xy -5.482516 2.806739) (xy -5.941136 2.437196)
+				(xy -6.832549 1.94563) (xy -7.239789 1.745747) (xy -8.888492 0.795645) (xy -10.070493 -0.266357)
+				(xy -10.845914 -1.502415) (xy -11.116067 -2.261698) (xy -11.215109 -3.227749) (xy -9.538718 -3.227749)
+				(xy -9.172235 -2.019384) (xy -8.355133 -0.946901) (xy -7.106999 -0.04063) (xy -5.447418 0.669102)
+				(xy -3.395979 1.151966) (xy -2.138006 1.307186) (xy -1.041811 1.386014) (xy -0.049939 1.425271)
+				(xy 0.633173 1.4171) (xy 0.661458 1.41479) (xy 1.362732 1.35379) (xy 2.34144 1.270323) (xy 3.090211 1.207249)
+				(xy 4.986595 0.894743) (xy 6.652247 0.319444) (xy 8.024985 -0.475467) (xy 9.042627 -1.446813) (xy 9.642991 -2.551413)
+				(xy 9.782029 -3.439584) (xy 9.526899 -4.801336) (xy 8.801563 -6.210935) (xy 7.648834 -7.586502)
+				(xy 7.577126 -7.656416) (xy 6.943902 -8.241512) (xy 6.47872 -8.621917) (xy 6.289401 -8.714749) (xy 6.131476 -8.422166)
+				(xy 5.843079 -7.865002) (xy 5.81252 -7.805209) (xy 5.405068 -7.237013) (xy 4.818185 -6.981669) (xy 4.403232 -6.928136)
+				(xy 3.448291 -6.994418) (xy 2.767208 -7.258865) (xy 2.167936 -7.603706) (xy 1.906619 -7.590273)
+				(xy 1.916115 -7.200753) (xy 1.952861 -7.042821) (xy 1.970944 -6.234338) (xy 1.726082 -5.373531)
+				(xy 1.300498 -4.69213) (xy 1.047897 -4.492332) (xy 0.256399 -4.273976) (xy -0.703931 -4.26385) (xy -1.518456 -4.462498)
+				(xy -1.568607 -4.487806) (xy -2.09355 -5.017236) (xy -2.461625 -5.83363) (xy -2.581111 -6.698815)
+				(xy -2.538473 -7.006323) (xy -2.48223 -7.527006) (xy -2.704656 -7.623778) (xy -3.238029 -7.307837)
+				(xy -3.291716 -7.267628) (xy -3.900335 -7.004894) (xy -4.702258 -6.88067) (xy -4.791002 -6.879167)
+				(xy -5.590083 -6.990054) (xy -6.147728 -7.40431) (xy -6.30399 -7.603022) (xy -6.831281 -8.326877)
+				(xy -7.738582 -7.364858) (xy -8.841478 -5.930815) (xy -9.434994 -4.541669) (xy -9.538718 -3.227749)
+				(xy -11.215109 -3.227749) (xy -11.268163 -3.74523) (xy -10.96126 -5.313631) (xy -10.235929 -6.877274)
+				(xy -9.132741 -8.346529) (xy -8.845605 -8.607078) (xy -5.78827 -8.607078) (xy -5.683661 -8.153676)
+				(xy -5.660235 -8.091432) (xy -5.296052 -7.785511) (xy -4.66032 -7.67692) (xy -3.972814 -7.766474)
+				(xy -3.453307 -8.054984) (xy -3.428482 -8.083169) (xy -2.915798 -8.371958) (xy -2.403898 -8.413898)
+				(xy -1.983613 -8.313681) (xy -1.783026 -8.042005) (xy -1.722574 -7.448212) (xy -1.719792 -7.118522)
+				(xy -1.643407 -6.282606) (xy -1.451391 -5.621306) (xy -1.356666 -5.464876) (xy -0.741863 -5.08829)
+				(xy 0.022364 -5.066715) (xy 0.705896 -5.38643) (xy 0.900056 -5.599443) (xy 1.169714 -6.311556) (xy 1.143679 -7.319235)
+				(xy 1.06496 -8.03091) (xy 1.142774 -8.363305) (xy 1.457671 -8.460824) (xy 1.783723 -8.466667) (xy 2.465914 -8.342063)
+				(xy 2.910416 -8.069792) (xy 3.434251 -7.748046) (xy 4.124559 -7.664569) (xy 4.766931 -7.807686)
+				(xy 5.146958 -8.165719) (xy 5.156203 -8.19209) (xy 5.197443 -8.881343) (xy 4.810201 -9.440154) (xy 3.957605 -9.903772)
+				(xy 3.066263 -10.189971) (xy 1.013297 -10.534918) (xy -1.109826 -10.517771) (xy -3.121762 -10.150111)
+				(xy -4.304717 -9.719211) (xy -5.18185 -9.290112) (xy -5.648684 -8.952645) (xy -5.78827 -8.607078)
+				(xy -8.845605 -8.607078) (xy -7.824398 -9.533729) (xy -5.576949 -10.930488) (xy -3.214395 -11.844752)
+				(xy -0.794897 -12.278751)
+			)
+			(stroke
+				(width 0)
+				(type solid)
+			)
+			(fill yes)
+			(layer "F.SilkS")
+		)
+		(embedded_fonts no)
 	)
 	(footprint "MX_Hotswap:MX-Hotswap-2.25U"

Commit message: Via stitching ground planes
Parts:
- moved D51 29.5 mm to (178.7, 129.6)
- moved D53 29.5 mm to (216.8, 129.6)
- moved D56 29.5 mm to (281.1, 129.5)
- moved J1 29.5 mm to (137.6, 143.0)
- moved SW52 29.5 mm to (173.1, 124.7)
- moved SW55 29.5 mm to (230.3, 124.7)
- moved SW64 29.5 mm to (227.9, 143.8)
- moved SW65 29.5 mm to (251.7, 143.8)
- moved SW68 29.5 mm to (320.8, 143.8)
- moved D2 29.5 mm to (59.6, 72.2)
- moved D3 29.5 mm to (78.7, 72.2)
- moved D45 29.5 mm to (52.5, 129.5)
- moved D46 29.5 mm to (83.4, 129.5)
- moved D47 29.5 mm to (102.5, 129.5)
- moved D48 29.5 mm to (121.5, 129.5)
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Routing:
- added copper zone on B.Cu, net GND

Commit message: More vias
Parts:
- moved D45 39.5 mm to (46.3, 90.5)
- moved D46 39.5 mm to (77.3, 90.5)
- moved D47 39.5 mm to (96.3, 90.5)
- moved D48 39.5 mm to (115.4, 90.5)
- moved D49 39.5 mm to (134.4, 90.5)
- moved D50 39.5 mm to (153.5, 90.5)
- moved D51 39.5 mm to (172.5, 90.5)
- moved D52 39.5 mm to (191.6, 90.5)
- moved D53 39.5 mm to (210.6, 90.5)
- moved D54 39.5 mm to (229.7, 90.5)
- moved D55 39.5 mm to (248.7, 90.5)
- moved D56 39.5 mm to (274.9, 90.5)
- moved D58 39.5 mm to (320.2, 90.5)
- moved G*** 39.5 mm to (116.4, 101.5)
- moved R6 39.5 mm to (192.4, 96.5)
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Routing:
- net GND: track 253.0 -> 260.3 mm, vias 5 -> 48
Other:
- outline, holes or cut-outs redrawn

Commit message: Update USB-C shield
Parts:
- added FB1: 60@100MHz, Inductor_SMD:L_0805_2012Metric_Pad1.05x1.20mm_HandSolder, B.Cu at (179.3, 20.4)
Connections:
- J3 pad SH1: GND -> GNDREF
- J3 pad SH2: GND -> GNDREF
- J3 pad SH3: GND -> GNDREF
- J3 pad SH4: GND -> GNDREF
Routing:
- net GND: track 260.3 -> 239.3 mm, vias 48 -> 46
- net GNDREF: track 0.00 -> 12.9 mm, vias 0 -> 6
- net RESET: vias 4 -> 6
- added copper zone on B.Cu, net GNDREF
- added copper zone on F.Cu, net GNDREF

Commit message: Added manufacturing files
Parts:
- moved D15 17.4 mm to (332.7, 45.1)
- moved D28 17.4 mm to (285.3, 64.4)
- moved D29 17.4 mm to (309.1, 64.3)
- moved D30 17.4 mm to (332.9, 64.3)
- moved D44 17.4 mm to (332.9, 83.3)
- moved D58 17.4 mm to (332.9, 102.4)
- moved SW67 17.4 mm to (308.3, 116.7)
- moved D67 17.4 mm to (332.9, 121.4)
- moved SW58 17.4 mm to (308.3, 97.6)
- moved SW66 17.4 mm to (289.2, 116.7)
- moved C1 17.4 mm to (196.4, 107.5)
- moved C4 17.4 mm to (204.2, 112.2)
- moved C7 17.4 mm to (210.0, 115.9)
- moved C8 17.4 mm to (194.5, 106.7)
- moved D10 17.4 mm to (218.4, 45.1)
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