File: keyboard_v0.kicad_sch (KiCad schematic)
At the start: 21 parts, among them J1 AVR-ISP-6, J3 UJ20-C-H-G-SMT-1-P16-TR, SW1 SW_RESET, U1 ATmega32U4-A, U2 USBLC6-2P6, Y1 Crystal_GND24_Small

Commit message: Update USB-C shield
Parts:
- added FB1: 60@100MHz, Inductor_SMD:L_0805_2012Metric_Pad1.05x1.20mm_HandSolder, symbol Device:FerriteBead_Small
Connections:
- net GND: now also FB1.2; no longer J3.SH1 (SHIELD), J3.SH2 (SHIELD), J3.SH3 (SHIELD), J3.SH4 (SHIELD)
- new net GNDREF: FB1.1, J3.SH1 (SHIELD), J3.SH2 (SHIELD), J3.SH3 (SHIELD), J3.SH4 (SHIELD)

Commit message: Added fab files
Parts:
- R6: value R_Small -> 10k
Changed lines of the file:
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@@
 			)
 		)
-		(property "Value" "R_Small"
+		(property "Value" "10k"
 			(at 106.68 110.4899 0)
 			(show_name no)
